Commit message: Refactor rt_controller_main into reusable function, add URDF-to-MJCF converter, fix mesh paths
- Extract rt_controller_main logic into RtControllerMain() in rt_controller_main_impl.cpp
  to eliminate duplication between generic and ur5e-specific entry points
- Use --whole-archive linking for demo controllers, removing ForceDemoControllerRegistration()
- Add urdf_to_mjcf tool (rtc_tools) to convert URDF/XACRO files to MuJoCo MJCF XML
  with automatic package:// URI resolution and xacro argument support
- Fix ur5e.urdf mesh paths: meshes/ur5e/{visual,collision}/ -> meshes/{visual,collision}/

Co-Authored-By: Claude Opus 4.6 (1M context) <noreply@anthropic.com>

File: ur5e_description/robots/ur5e/urdf/ur5e.urdf (robot description, URDF)
Before this commit: robot ur5e, 13 links, 12 joints
Links:
- link base_link_inertia: geometry collision mesh filename=package://ur5e_description/robots/ur5e/meshes/collision/bas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; visual mesh filename=package://ur5e_description/robots/ur5e/meshes/visual/base.d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
- link forearm_link: geometry collision mesh filename=package://ur5e_description/robots/ur5e/meshes/collision/for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; visual mesh filename=package://ur5e_description/robots/ur5e/meshes/visual/forear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
- link shoulder_link: geometry collision mesh filename=package://ur5e_description/robots/ur5e/meshes/collision/sho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; visual mesh filename=package://ur5e_description/robots/ur5e/meshes/visual/should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
- link upper_arm_link: geometry collision mesh filename=package://ur5e_description/robots/ur5e/meshes/collision/upp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; visual mesh filename=package://ur5e_description/robots/ur5e/meshes/visual/uppera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
- link wrist_1_link: geometry collision mesh filename=package://ur5e_description/robots/ur5e/meshes/collision/wri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; visual mesh filename=package://ur5e_description/robots/ur5e/meshes/visual/wrist1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
- link wrist_2_link: geometry collision mesh filename=package://ur5e_description/robots/ur5e/meshes/collision/wri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; visual mesh filename=package://ur5e_description/robots/ur5e/meshes/visual/wrist2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
- link wrist_3_link: geometry collision mesh filename=package://ur5e_description/robots/ur5e/meshes/collision/wri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; visual mesh filename=package://ur5e_description/robots/ur5e/meshes/visual/wrist3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
