Commit message: refactor!: rename ur5e_description -> robot_descriptions, robot-agnostic data hub
The package is no longer UR5e-specific; rename to reflect that it is a
multi-robot data hub.  One subdirectory per robot/hand under robots/,
with no C++ code or framework deps.  UR5e + the custom hand are first
tenants; allegro / leap / schunk / iiwa7 etc. drop in later as additional
robots/<name>/ subdirectories.

- Subdirectory rename: robots/hand_tmp/ -> robots/assm_v1/,
  robots/ur5e_hand_tmp/ -> robots/ur5e_assm_v1/ (drop _tmp suffix).
- README rewritten: §1 declares the package robot-agnostic and explains
  how new robots are added without touching its build files.
- repo_scripts/get_base_packages now contains robot_descriptions
  (it is robot-agnostic); get_robot_packages drops it.
- All dependents (ur5e_bringup, rtc_digital_twin, rtc_tools,
  rtc_mujoco_sim, rtc_controller_manager) updated: package.xml,
  CMakeLists.txt, *.yaml, *.launch.py, *.md, mesh package:// URIs,
  and the combined urdf.xacro xacro:include filenames.
- CLAUDE.md §1 split: ur5e_* now (3), robot_descriptions (1).  Total
  package count unchanged at 20.

Note: install/ur5e_description from previous workspace state is now
stale; remove with `rm -rf install/ur5e_description build/ur5e_description`
or `./build.sh --clean full` to silence colcon override warnings.

Co-Authored-By: Claude Opus 4.7 (1M context) <noreply@anthropic.com>

File: robot_descriptions/robots/ur5e/urdf/ur5e.urdf (robot description, URDF)
Before this commit: robot ur5e, 13 links, 12 joints
Links:
- link base_link_inertia: geometry collision mesh filename=package://robot_descriptions/robots/ur5e/meshes/collision/b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; visual mesh filename=package://robot_descriptions/robots/ur5e/meshes/visual/base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
- link forearm_link: geometry collision mesh filename=package://robot_descriptions/robots/ur5e/meshes/collision/f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; visual mesh filename=package://robot_descriptions/robots/ur5e/meshes/visual/fore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
- link shoulder_link: geometry collision mesh filename=package://robot_descriptions/robots/ur5e/meshes/collision/s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; visual mesh filename=package://robot_descriptions/robots/ur5e/meshes/visual/shou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
- link upper_arm_link: geometry collision mesh filename=package://robot_descriptions/robots/ur5e/meshes/collision/u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; visual mesh filename=package://robot_descriptions/robots/ur5e/meshes/visual/uppe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
- link wrist_1_link: geometry collision mesh filename=package://robot_descriptions/robots/ur5e/meshes/collision/w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; visual mesh filename=package://robot_descriptions/robots/ur5e/meshes/visual/wris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
- link wrist_2_link: geometry collision mesh filename=package://robot_descriptions/robots/ur5e/meshes/collision/w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; visual mesh filename=package://robot_descriptions/robots/ur5e/meshes/visual/wris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
- link wrist_3_link: geometry collision mesh filename=package://robot_descriptions/robots/ur5e/meshes/collision/w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; visual mesh filename=package://robot_descriptions/robots/ur5e/meshes/visual/wris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

File: robot_descriptions/robots/ur5e_assm_v1/urdf/ur5e_with_hand.urdf.xacro (robot description, xacro)
@@ -7,7 +7,7 @@
 <robot xmlns:xacro="http://www.ros.org/wiki/xacro" name="ur5e_with_hand">
   <!-- UR5e base robot (pre-generated URDF, included as-is) -->
-  <xacro:include filename="$(find ur5e_description)/robots/ur5e/urdf/ur5e.urdf"/>
+  <xacro:include filename="$(find robot_descriptions)/robots/ur5e/urdf/ur5e.urdf"/>
   <!-- Custom Hand model -->
-  <xacro:include filename="$(find ur5e_description)/robots/hand_tmp/urdf/hand.urdf.xacro"/>
+  <xacro:include filename="$(find robot_descriptions)/robots/assm_v1/urdf/hand.urdf.xacro"/>
   <!-- Attach hand to tool0 -->
   <joint name="tool0_to_hand" type="fixed">
