Commit message: test(multi-pkg): Move the p1b and G1 fixtures onto the test models
Every fixture that opened robot_descriptions/robots/ur5e_p1b/ (the
vendored proto_1b, #457) or hand_description's G1 now opens the
profile's test model from p1b_surrogate_models.hpp; the profile's
sub-models, tree models, extra frames and devices are still read from
the shipped YAML. The G1 cases lose their RTC_SKIP_IF_PACKAGE_MISSING
guards, optional_package.hpp goes with them, and the vendored proto_1b
copy is removed.

The pilot fixture's robot.urdf is regenerated from the surrogate and
make_fixture.py writes it that way. The rtc_tools goldens (287 cases)
are unchanged: they read the arm, the palm frame and the link names,
which the surrogate keeps.

Two integrated_bringup cases pin numbers of the real hand and fail on
this commit; the next two re-pin them (PROC-6).

Refs: #952

Co-Authored-By: Claude Opus 5.5 <noreply@anthropic.com>

File: rtc_tools/test/data/catching_pilot_260924_1218/robot.urdf (robot description, URDF)
Before this commit: robot ur5e_with_proto_1b, 49 links, 48 joints
Links:
- link l_index_dip_link: mass 0.06404 -> 0.05; geometry collision box size=0.014 0.046 0.014; visual box size=0.014 0.046 0.014
- link l_index_mcp_link: mass 0.065 -> 0.02; geometry collision box size=0.014 0.014 0.014; visual box size=0.014 0.014 0.014
- link l_index_pip_linkage_a: mass 0.00143 -> 0.003; geometry collision box size=0.006 0.026 0.006; visual box size=0.006 0.026 0.006
- link l_index_pip_linkage_b: mass 0.00645 -> 0.012; geometry collision box size=0.014 0.026 0.014; visual box size=0.014 0.026 0.014
- link l_index_tip_link: mass 0.01259 -> 0.015; geometry collision box size=0.014 0.022 0.014; visual box size=0.014 0.022 0.014
- link l_middle_dip_a_link: mass 0.00143 -> 0.003; geometry collision box size=0.006 0.026 0.006; visual box size=0.006 0.026 0.006
- link l_middle_dip_b_link: mass 0.00745 -> 0.012; geometry collision box size=0.014 0.026 0.014; visual box size=0.014 0.026 0.014
- link l_middle_mcp_link: mass 0.06404 -> 0.05; geometry collision box size=0.014 0.05 0.014; visual box size=0.014 0.05 0.014
- link l_middle_tip_link: mass 0.01259 -> 0.015; geometry collision box size=0.014 0.022 0.014; visual box size=0.014 0.022 0.014
- link l_palm_link: mass 0.7679600000000001 -> 0.55; geometry collision box size=0.09 0.12 0.03; visual box size=0.09 0.12 0.03
- link l_ring_dip_linkage_a: mass 0.00143 -> 0.003; geometry collision box size=0.006 0.023000000000000007 0.006; visual box size=0.006 0.023000000000000007 0.006
- link l_ring_dip_linkage_b: mass 0.00783 -> 0.01; geometry collision box size=0.014 0.024000000000000007 0.014; visual box size=0.014 0.024000000000000007 0.014
- link l_ring_pip_linkage_a: mass 0.00245 -> 0.004; geometry collision box size=0.006 0.041999999999999996 0.006; visual box size=0.006 0.041999999999999996 0.006
- link l_ring_pip_linkage_b: mass 0.02015 -> 0.04; geometry collision box size=0.014 0.045 0.014; visual box size=0.014 0.045 0.014
- link l_ring_tip_link: mass 0.01259 -> 0.015; geometry collision box size=0.014 0.022 0.014; visual box size=0.014 0.022 0.014
- link l_thumb_cmc_link_a: mass 0.01386 -> 0.015; geometry collision box size=0.016 0.014 0.014; visual box size=0.016 0.014 0.014
- link l_thumb_cmc_link_b: mass 0.03 -> 0.025; geometry collision box size=0.02 0.014 0.014; visual box size=0.02 0.014 0.014
- link l_thumb_dip_link_a: mass 0.00143 -> 0.003; geometry collision box size=0.026 0.006 0.006; visual box size=0.026 0.006 0.006
- link l_thumb_dip_link_b: mass 0.00745 -> 0.012; geometry collision box size=0.026 0.014 0.014; visual box size=0.026 0.014 0.014
- link l_thumb_mcp_link: mass 0.09931 -> 0.06; geometry collision box size=0.04 0.014 0.014; visual box size=0.04 0.014 0.014
- link l_thumb_tip_link: mass 0.01259 -> 0.015; geometry collision box size=0.022 0.014 0.014; visual box size=0.022 0.014 0.014
Joints:
- removed joint tool0_to_proto_1b
- added joint tool0_to_p1b_surrogate: type fixed, parent tool0, child base_adapter, origin xyz=0 0 0 rpy=0 0 0
- joint index_dip_a_joint_passive: origin xyz=8.611e-05 0.0499993 -0.00078834 rpy=0 0 0 -> xyz=0.0 0.046 -0.004 rpy=0 0 0
- joint index_dip_fe_joint: limit lower=-1.5707963267948963 upper=0.0 effort=3.0 velocity=10.384 -> lower=-1.5707963267948966 upper=0.0 effort=3.0 velocity=10.384; origin xyz=0.0 0.0450137 0.00221116 rpy=0 0 0 -> xyz=0.0 0.046 0.0 rpy=0 0 0
- joint index_mcp_aa_joint: limit lower=-0.122173048 upper=0.296705973 effort=3.0 velocity=10.384 -> lower=-0.34906585 upper=0.523598776 effort=3.0 velocity=10.384; origin xyz=0.031 0.1358 -0.00204608 rpy=0 0 0 -> xyz=0.026 0.125 0.0 rpy=0 0 0
- joint index_mcp_fe_joint: limit lower=-1.5707963267948963 upper=0.0 effort=3.0 velocity=10.384 -> lower=-1.5707963267948966 upper=0.0 effort=3.0 velocity=10.384; origin xyz=0.0 0.0 0.0 rpy=0 0 0 -> xyz=0 0 0 rpy=0 0 0
- joint index_pip_a_joint_passive: origin xyz=-8.611e-05 0.0207689 0.0109956 rpy=0 0 0 -> xyz=0.0 0.026 -0.004 rpy=0 0 0
- joint index_pip_b_joint_constraint_ab: origin xyz=0.0 0.00025994 -0.00999662 rpy=0 0 0 -> xyz=0.0 0.0 0.008 rpy=0 0 0
- joint index_pip_b_joint_constraint_ba: origin xyz=0.0 0.0260144 -0.00200051 rpy=0 0 0 -> xyz=0.0 0.026 0.0 rpy=0 0 0
- joint index_tip_bracket_joint_fixed: origin xyz=0.0 0.0170877 -0.00354701 rpy=0 0 1.570796327 -> xyz=0.0 0.022 0.006 rpy=0 0 1.5707963267948966
- joint middle_dip_a_joint_passive: origin xyz=-0.00552899 0.05 -0.003 rpy=0 0 0 -> xyz=0.0 0.05 -0.004 rpy=0 0 0
- joint middle_dip_fe_joint: limit lower=-1.5707963267948963 upper=0.0 effort=3.0 velocity=10.384 -> lower=-1.5707963267948966 upper=0.0 effort=3.0 velocity=10.384; origin xyz=-0.00552899 0.0450144 0.0 rpy=0 0 0 -> xyz=0.0 0.05 0.0 rpy=0 0 0
- joint middle_mcp_fe_joint: limit lower=-1.5707963267948963 upper=0.0 effort=3.0 velocity=10.384 -> lower=-1.5707963267948966 upper=0.0 effort=3.0 velocity=10.384; origin xyz=0.00552899 0.1513 0.0 rpy=0 0 0 -> xyz=0.0 0.13 0.0 rpy=0 0 0
- joint middle_pip_a_joint_passive: origin xyz=0.0 0.0207689 0.0109956 rpy=0 0 0 -> xyz=0.0 0.026 -0.004 rpy=0 0 0
- joint middle_pip_b_joint_constraint_ab: origin xyz=0.0 0.00025995 -0.00999663 rpy=0 0 0 -> xyz=0.0 0.0 0.008 rpy=0 0 0
- joint middle_pip_b_joint_constraint_ba: origin xyz=0.0 0.0260144 -0.00200101 rpy=0 0 0 -> xyz=0.0 0.026 0.0 rpy=0 0 0
- joint middle_tip_bracket_joint_fixed: origin xyz=0.0 0.0170877 -0.00354701 rpy=0 0 1.570796327 -> xyz=0.0 0.022 0.006 rpy=0 0 1.5707963267948966
- joint ring_dip_a_joint_passive: origin xyz=-0.00546788 0.051 -0.004 rpy=0 0 0 -> xyz=0 0.045 -0.004 rpy=0 0 0
- joint ring_dip_b_joint_constraint_ab: origin xyz=-8.611e-05 -0.00234447 -0.00712415 rpy=0 0 0 -> xyz=0 0.0010000000000000009 0.014 rpy=0 0 0
- joint ring_dip_b_joint_constraint_ba: origin xyz=-0.00555399 0.045 0.0 rpy=0 0 0 -> xyz=0 0.045 0 rpy=0 0 0
- joint ring_dip_b_joint_passive: origin xyz=0.0 0.0417709 0.0121426 rpy=0 0 0 -> xyz=0 0.041999999999999996 -0.012 rpy=0 0 0
- joint ring_mcp_a_joint_passive: origin xyz=-0.0309389 0.141374 -0.00501848 rpy=0 0 0 -> xyz=-0.026 0.124 -0.002 rpy=0 0 0
- joint ring_mcp_fe_joint: limit lower=-1.5707963267948963 upper=0.0 effort=3.0 velocity=10.384 -> lower=-1.5707963267948966 upper=0.0 effort=3.0 velocity=10.384; origin xyz=-0.025471 0.1358 0.0 rpy=0 0 0 -> xyz=-0.026 0.122 0.0 rpy=0 0 0
- joint ring_pip_a_joint_passive: origin xyz=-8.611e-05 0.0197052 0.0128046 rpy=0 0 0 -> xyz=0 0.023000000000000007 -0.004 rpy=0 0 0
- joint ring_pip_b_joint_constraint_ab: origin xyz=0.0 0.00034452 -0.00999407 rpy=0 0 0 -> xyz=0 0.0 0.008 rpy=0 0 0
- joint ring_pip_b_joint_constraint_ba: origin xyz=-8.611e-05 0.0237052 -0.00831364 rpy=0 0 0 -> xyz=0 0.024000000000000007 0.014 rpy=0 0 0
- joint ring_tip_bracket_joint_fixed: origin xyz=0.0 0.0170877 -0.00354701 rpy=0 0 1.570796327 -> xyz=0 0.022 0.006 rpy=0 0 1.5707963267948966
- joint thumb_cmc_aa_joint: limit lower=0.0 upper=2.35619449 effort=3.0 velocity=10.384 -> lower=0.0 upper=2.356194487 effort=3.0 velocity=10.384; origin xyz=0.0155 0.0478947 0.0345 rpy=0 0 0 -> xyz=0.038 0.035 0.018 rpy=0 0 0
- joint thumb_cmc_fe_joint: origin xyz=0.0 0.0198053 0.0 rpy=0 0 0 -> xyz=0.016 0 0 rpy=0 0 0
- joint thumb_dip_a_joint_passive: origin xyz=0.00186253 0.0610706 -0.00093889 rpy=0 0 0 -> xyz=0.04 -0.004 0.0 rpy=0 0 0
- joint thumb_dip_fe_joint: limit lower=-1.5707963267948963 upper=0.0 effort=3.0 velocity=10.384 -> lower=-1.5707963267948966 upper=0.0 effort=3.0 velocity=10.384; origin xyz=-0.00113798 0.0560562 -0.001 rpy=0 0 0 -> xyz=0.04 0.0 0.0 rpy=0 0 0
- joint thumb_mcp_joint: origin xyz=0.020002 0.0136114 0.0 rpy=0 0 -0.7853981633974485 -> xyz=0.02 0 0 rpy=0 0 0
- joint thumb_pip_a_joint_passive: origin xyz=-0.0109973 0.020768 -8.611e-05 rpy=0 0 0 -> xyz=0.026 -0.004 0.0 rpy=0 0 0
- joint thumb_pip_b_joint_constraint_ab: origin xyz=0.00999731 0.000232023 0.0 rpy=0 0 0 -> xyz=0.0 0.008 0.0 rpy=0 0 0
- joint thumb_pip_b_joint_constraint_ba: origin xyz=0.00200051 0.0260144 -2.5e-05 rpy=0 0 0 -> xyz=0.026 0.0 0.0 rpy=0 0 0
- joint thumb_tip_bracket_joint_fixed: origin xyz=0.00354701 0.0170877 0.0 rpy=-1.570796327 0 1.570796327 -> xyz=0.022 0.006 0.0 rpy=-1.5707963267948966 0 1.5707963267948966
